Commit message: Nicholas' configuration

File: dvrk_description/psm/psm_modified.urdf (robot description, URDF)
Before this commit: robot master, 11 links, 10 joints
Joints:
- joint psm_tool_yaw_joint: origin xyz=0.0091 0 0 rpy=0 -1.5708 3.1416 -> xyz=0.0091 0 0 rpy=1.5708 -1.5708 3.1416
- joint tool_tip: origin xyz=0 0 0.0102 rpy=0 0 0 -> xyz=0 0.0102 0 rpy=0 0 0

Commit message: Hybrid configuration (correct with dvrk documentation)

File: dvrk_description/psm/psm_modified.urdf (robot description, URDF)
Before this commit: robot master, 11 links, 10 joints
Joints:
- joint tool_tip: origin xyz=0 0.0102 0 rpy=0 0 0 -> xyz=0 0.0102 0 rpy=-1.5707 1.5707 0
